Commit message: working model of casadi based pinoccio dynamic symbolic function, which is very useful for cast ioptimization in casadi

File: model/double_pend.urdf (robot description, URDF)
Before this commit: robot cart_double_pendulum, 5 links, 4 joints
Links:
- link cart: geometry visual box size=0.1 0.1 0.05
